Commit message: AM-591/am-configuration

File: launch/include/config/robot.urdf.xacro (robot description, xacro)
@@ -27,3 +27,9 @@
     <origin xyz="0 0 0" rpy="0 0 0" />
   </joint>
+  <link name="body_FLU"> </link>
+  <joint name="body_FLU_joint" type="fixed">
+    <parent link="chassis_link" />
+    <child link="body_FLU" />
+    <origin xyz="0 0 0" rpy="0 0 0" />
+  </joint>
 </robot>
